File: eagle_files/current_only/current_only.sch (EAGLE design)
At the start: 6 parts, among them J1 ST-PJ-312, J2 PJ-393

Commit message: d
Parts:
- removed J2: PJ-393, Seeed-Connector:AUDIO-JACK-PJ-393(8P-SMD)
- added CN1: 3p-2.54, Seeed-Connector:DIP-BLACK-MALE-HEADER-VERT(3P-2.54)
Connections:
- net +5V: now also CN1.P$2
- net GND: now also CN1.P$1
- net N$1: now also J1.RS; no longer J2.GND
- net N$2: now also CN1.P$3, J1.COM2; no longer J2.MIC
Other:
- moved on the sheet: J1
Changed lines of the file:
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@@
 <setting verticaltext="up"/>
 </settings>
-<grid distance="0.1" unitdist="inch" unit="inch" style="lines" multiple="1" display="no" altdistance="0.01" altunitdist="inch" altunit="inch"/>
+<grid distance="0.1" unitdist="inch" unit="inch" style="dots" multiple="1" display="yes" altdistance="0.01" altunitdist="inch" altunit="inch"/>
 <layers>
 <layer number="1" name="Top" color="4" fill="1" visible="no" active="no"/>
@@
 <part name="J1" library="Seeed-Connector" deviceset="AUDIO-JACK-6P-SMD(ST-PJ-312)" device="" value="ST-PJ-312"/>
 <part name="P+1" library="supply1" library_urn="urn:adsk.eagle:library:371" deviceset="+5V" device=""/>
-<part name="J2" library="Seeed-Connector" deviceset="AUDIO-JACK-PJ-393(8P-SMD)" device="" value="PJ-393"/>
+<part name="CN1" library="Seeed-Connector" deviceset="DIP-BLACK-MALE-HEADER-VERT(3P-2.54)" device="" value="3p-2.54"/>
+<part name="P+2" library="supply1" library_urn="urn:adsk.eagle:library:371" deviceset="+5V" device=""/>
+<part name="GND2" library="supply1" library_urn="urn:adsk.eagle:library:371" deviceset="GND" device=""/>
 </parts>
 <sheets>
@@
 <plain>
 <text x="55.88" y="68.58" size="1.778" layer="91">A1</text>
+<text x="68.58" y="60.96" size="1.778" layer="91">A1</text>
 </plain>
 <instances>
@@
 <instance part="R3" gate="G$1" x="17.78" y="60.96" rot="R90"/>
 <instance part="GND1" gate="1" x="55.88" y="38.1" rot="R90"/>
-<instance part="J1" gate="G$1" x="-20.32" y="35.56" rot="R180"/>
+<instance part="J1" gate="G$1" x="-2.54" y="63.5" rot="R180"/>
 <instance part="P+1" gate="1" x="60.96" y="71.12" rot="R270"/>
-<instance part="J2" gate="G$1" x="-10.16" y="63.5"/>
+<instance part="CN1" gate="G$1" x="58.42" y="55.88" rot="R180"/>
+<instance part="P+2" gate="1" x="73.66" y="55.88" rot="R270"/>
+<instance part="GND2" gate="1" x="71.12" y="50.8" rot="R90"/>
 </instances>
 <busses>
@@
 <wire x1="17.78" y1="53.34" x2="17.78" y2="55.88" width="0.1524" layer="91"/>
 <junction x="17.78" y="53.34"/>
-<wire x1="17.78" y1="53.34" x2="0" y2="53.34" width="0.1524" layer="91"/>
-<pinref part="J2" gate="G$1" pin="GND"/>
-<wire x1="0" y1="53.34" x2="0" y2="54.61" width="0.1524" layer="91"/>
+<wire x1="17.78" y1="53.34" x2="6.35" y2="53.34" width="0.1524" layer="91"/>
+<pinref part="J1" gate="G$1" pin="RS"/>
 </segment>
 </net>
@@
 <pinref part="C1" gate="G$1" pin="+"/>
 <wire x1="30.48" y1="38.1" x2="30.48" y2="52.07" width="0.1524" layer="91"/>
+<junction x="53.34" y="38.1"/>
+</segment>
+<segment>
+<pinref part="CN1" gate="G$1" pin="P$1"/>
+<pinref part="GND2" gate="1" pin="GND"/>
+<wire x1="66.04" y1="52.07" x2="68.58" y2="50.8" width="0.1524" layer="91"/>
+<junction x="68.58" y="50.8"/>
 </segment>
 </net>
@@
 <wire x1="17.78" y1="66.04" x2="17.78" y2="68.58" width="0.1524" layer="91"/>
 <wire x1="17.78" y1="68.58" x2="55.88" y2="68.58" width="0.1524" layer="91"/>
-<wire x1="17.78" y1="68.58" x2="17.78" y2="73.66" width="0.1524" layer="91"/>
+<wire x1="17.78" y1="68.58" x2="17.78" y2="76.2" width="0.1524" layer="91"/>
 <junction x="17.78" y="68.58"/>
-<pinref part="J2" gate="G$1" pin="MIC"/>
-<wire x1="0" y1="73.66" x2="17.78" y2="73.66" width="0.1524" layer="91"/>
+<pinref part="J1" gate="G$1" pin="COM2"/>
+<wire x1="-13.97" y1="73.66" x2="-11.43" y2="76.2" width="0.1524" layer="91"/>
+<wire x1="-11.43" y1="76.2" x2="17.78" y2="76.2" width="0.1524" layer="91"/>
+<junction x="55.88" y="68.58"/>
+<wire x1="55.88" y1="68.58" x2="55.88" y2="63.5" width="0.1524" layer="91"/>
+<wire x1="55.88" y1="63.5" x2="68.58" y2="63.5" width="0.1524" layer="91"/>
+<pinref part="CN1" gate="G$1" pin="P$3"/>
+<wire x1="66.04" y1="59.69" x2="67.31" y2="60.96" width="0.1524" layer="91"/>
+<wire x1="67.31" y1="60.96" x2="68.58" y2="60.96" width="0.1524" layer="91"/>
+<junction x="68.58" y="60.96"/>
+<wire x1="68.58" y1="63.5" x2="68.58" y2="60.96" width="0.1524" layer="91"/>
 </segment>
 </net>
@@
 <wire x1="43.18" y1="71.12" x2="58.42" y2="71.12" width="0.1524" layer="91"/>
 <pinref part="P+1" gate="1" pin="+5V"/>
+<junction x="58.42" y="71.12"/>
+</segment>
+<segment>
+<pinref part="CN1" gate="G$1" pin="P$2"/>
+<pinref part="P+2" gate="1" pin="+5V"/>
+<wire x1="71.12" y1="55.88" x2="66.04" y2="55.88" width="0.1524" layer="91"/>
+<junction x="71.12" y="55.88"/>
+<junction x="66.04" y="55.88"/>
 </segment>
 </net>
@@
 </drawing>
 <compatibility>
-<note version="6.3" minversion="6.2.2" severity="warning">
-Since Version 6.2.2 text objects can contain more than one line,
-which will not be processed correctly with this version.
-</note>
 <note version="8.2" severity="warning">
 Since Version 8.2, EAGLE supports online libraries. The ids
